File: Reg.sch (KiCad schematic (older format))
At the start: 40 parts, among them Q1 TIP41, Q2 TIP42, Q3 TIP35C, Q4 TIP35C, Q5 TIP35C, Q6 TIP35C, U1 LT6105, U2 NE5532, U3 NE5532

Commit message: Updates + Lot of routing
Connections:
- net I_Q3: now reaches Q3.3 (E), R14.2
- net I_Q4: now reaches Q4.3 (E), R15.2
- net I_Q5: now reaches Q5.3 (E), R16.2
- net I_Q6: now reaches Q6.3 (E), R17.2
Changed lines of the file:
@@
 	8400 3275 8100 3275
 Connection ~ 8100 3275
+Text Label 6825 850  0    60   ~ 0
+I_Q3
+Text Label 6850 1350 0    60   ~ 0
+I_Q4
+Text Label 6850 1850 0    60   ~ 0
+I_Q5
+Text Label 6850 2350 0    60   ~ 0
+I_Q6
 $EndSCHEMATC
