File: BypassCaps.sch (KiCad schematic (older format))
At the start: 8 parts

Commit message: Updates + Lot of routing
Parts:
- added C19, C20, C21, C22, C23: 100n, Capacitors_SMD:C_0805_HandSoldering, symbol C
Connections:
- net +3V3: now also C19.2
- net +5V: now also C12.2, C20.2, C21.2, C22.2, C23.2
- net -12V: no longer C11.1, C12.1
- net GND: now also C12.1, C19.1, C20.1, C21.1, C22.1, C23.1; no longer C11.2, C12.2
Other:
- note added: "U1 \nLT6105"
- note added: "U10\nFRAM"
- note added: "U2\nNE5532"
- note added: "U3\nNE5532"
- note added: "U4\nLM1117"
- note added: "U5\nTeensy"
- note added: "U7\nDAC I"
- note added: "U8\nDAC V"
- note added: "U9\nADC"
- moved on the sheet: C10, C11, C12, C13, C6, C7, C8, C9

Commit message: Finished routing
Connections:
- net -12V: now also C11.1
- net GND: now also C11.2
Changed lines of the file:
@@
 Wire Wire Line
 	8600 3300 8600 3225
+Wire Wire Line
+	4000 3650 4000 3800
+Wire Wire Line
+	4000 3350 4000 3250
 $EndSCHEMATC
