File: Regulator.kicad_pcb (KiCad board)
At the start: 2 copper layers, 160 x 7 mm, 86 parts, among them J1 +12V_IN, J10 LCD Header, J11 CONN_02X08, J2 RTN_12V, J3 -12V_IN, J4 PWR_IN, J5 PWR_IN_RTN, J6 PWR_OUT, J7 PWR_OUT_RTN, J8 JUMPER, J9 JUMPER, Q1 TIP41, Q2 TIP42, Q3 TIP35C, Q4 TIP35C, Q5 TIP35C, Q6 TIP35C, U1 LT6105, U10 MB85RC256V, U2 NE5532, U3 NE5532, U4 LM1117-5.0, U5 Teensy_3.2_NoProg, U6 REF2041, U7 DAC121C085, U8 DAC121C085, U9 ADS1115

Commit message: Finished routing
Parts:
- added J12: CONN_02X08, Connectors:IDC_Header_Straight_16pins, F.Cu at (167.4, 64.7)
- added REF**: 1pin, Connectors:1pin, F.Cu at (259.1, 101.6)
- added REF**: 1pin, Connectors:1pin, F.Cu at (259.1, 48.3)
- added REF**: 1pin, Connectors:1pin, F.Cu at (111.8, 48.3)
- added REF**: 1pin, Connectors:1pin, F.Cu at (111.8, 101.6)
- C1, C10, C11, C12, C13, C14, C16, C19, C2, C20, C21, C22, C23, C6, C7, C8, D1, D2, D3, D4, D5, R1, R10, R18, R19, R20, R21, R22, R23, R27, R4, R6, R9: moved to B.Cu
- J11: value CONN_02X08 -> CONN_01X07; footprint Connectors:IDC_Header_Straight_16pins -> Pin_Headers:Pin_Header_Straight_1x07_Pitch2.54mm
- moved J11 146.7 mm to (241.7, 94.2), turned to 90 degrees
- moved C9 135.9 mm to (153.2, 81.0), turned to 180 degrees
- moved C13 134.1 mm to (161.2, 71.8), turned to 270 degrees
- moved C21 118.9 mm to (164.6, 91.5), turned to 90 degrees
- moved C20 117.9 mm to (170.6, 91.7), turned to 90 degrees
- moved C4 105.8 mm to (136.2, 89.3)
- moved R13 105.7 mm to (141.4, 89.3), turned to 270 degrees
- moved U5 105.0 mm to (209.7, 84.7)
- moved C22 99.3 mm to (179.7, 84.5), turned to 270 degrees
- moved C5 94.8 mm to (143.6, 89.2), turned to 90 degrees
- moved C15 90.1 mm to (157.3, 67.9), turned to 180 degrees
- moved C23 87.9 mm to (191.2, 79.2)
- moved C12 84.0 mm to (211.1, 72.5), turned to 180 degrees
- moved C14 83.4 mm to (154.6, 73.7), turned to 90 degrees
- moved U4 79.6 mm to (155.3, 74.3)
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Connections:
- C11 pad 1: Net-(C11-Pad1) -> -12V
- C11 pad 2: Net-(C11-Pad2) -> GND
- J11 pad 1: GND -> Net-(J11-Pad1)
- J11 pad 2: +5V -> Net-(J11-Pad2)
- U5 pad 10: Net-(J10-Pad7) -> Net-(J11-Pad2)
- U5 pad 11: Net-(J10-Pad8) -> Net-(J11-Pad3)
- U5 pad 12: Net-(J10-Pad9) -> Net-(J11-Pad4)
- U5 pad 13: Net-(J10-Pad10) -> Net-(J11-Pad5)
- U5 pad 14: Net-(U5-Pad14) -> Net-(J11-Pad6)
- U5 pad 2: Net-(J11-Pad4) -> Net-(U10-Pad7)
- U5 pad 20: Net-(J11-Pad16) -> Net-(J12-Pad4)
- U5 pad 21: Net-(J11-Pad15) -> Net-(J11-Pad7)
- U5 pad 22: Net-(J11-Pad13) -> Net-(J12-Pad6)
- U5 pad 23: Net-(J11-Pad11) -> Net-(J12-Pad8)
- U5 pad 24: Net-(J11-Pad9) -> Net-(J12-Pad10)
- U5 pad 27: Net-(J11-Pad7) -> Net-(J12-Pad12)
- U5 pad 28: Net-(J11-Pad5) -> Net-(J12-Pad14)
- U5 pad 29: Net-(J11-Pad3) -> Net-(J12-Pad16)
- U5 pad 3: Net-(J11-Pad6) -> Net-(J10-Pad4)
- U5 pad 30: Net-(U10-Pad7) -> Net-(U5-Pad30)
- U5 pad 4: Net-(J11-Pad8) -> Net-(J10-Pad6)
- U5 pad 5: Net-(J11-Pad10) -> Net-(J10-Pad7)
- U5 pad 6: Net-(J11-Pad12) -> Net-(J10-Pad8)
- U5 pad 7: Net-(J11-Pad14) -> Net-(J10-Pad9)
- U5 pad 8: Net-(J10-Pad4) -> Net-(J10-Pad10)
- U5 pad 9: Net-(J10-Pad6) -> Net-(J11-Pad1)
- U9 pad 2: Net-(U5-Pad14) -> Net-(U5-Pad30)
Routing:
- net /Control/SCL: track 0.00 -> 114.6 mm, vias 0 -> 8
- net /Control/SDA: track 0.00 -> 108.3 mm, vias 0 -> 9
- net Net-(R27-Pad1): track 0.00 -> 92.2 mm, vias 0 -> 5
- net Net-(J12-Pad4): track 0.00 -> 79.4 mm
- net Net-(J12-Pad6): track 0.00 -> 71.7 mm
- net Net-(J12-Pad8): track 0.00 -> 66.1 mm
- net Net-(J12-Pad10): track 0.00 -> 60.4 mm
- net Net-(R26-Pad1): track 0.00 -> 51.8 mm, vias 0 -> 4
- net Net-(J12-Pad12): track 0.00 -> 49.4 mm
- net Net-(U5-Pad30): track 0.00 -> 48.4 mm, vias 0 -> 2
- net Net-(J12-Pad14): track 0.00 -> 44.2 mm
- net /Control/Iset: track 13.9 -> 55.4 mm, vias 2 -> 4
- net Net-(J12-Pad16): track 0.00 -> 38.3 mm
- net +5V: track 0.00 -> 37.1 mm, vias 0 -> 8
- net +3V3: track 0.00 -> 35.3 mm
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Other:
- board size 160 x 7 mm -> 158 x 64 mm
